File: regulator/regulator.kicad_sch (KiCad schematic)
At the start: 10 parts, among them J1 Conn_01x02, J2 Conn_01x02, U1 TPS79333-EP

Commit message: pcb layout (connection errors)
Parts:
- C2: value 0.01uF -> 2.2uF
- C3: value 2.2uF -> 0.01uF
Changed lines of the file:
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@@
-	(wire
-		(pts
-			(xy 190.5 93.98) (xy 190.5 92.71)
-		)
-		(stroke
-			(width 0)
-			(type default)
-		)
-	)
 	(wire
 		(pts
@@
 			)
 		)
-		(property "Value" "0.01uF"
+		(property "Value" "2.2uF"
 			(at 163.83 101.5999 0)
 			(effects
@@
 			)
 		)
-		(property "Value" "2.2uF"
+		(property "Value" "0.01uF"
 			(at 152.4 107.9499 0)
 			(effects
